Commit message: Add a custom mesh to the robot urdf - change in cmake - urdf and launch

File: src/gazebo_pg/urdf/example_gazebo.xacro (robot description, xacro)
@@ -17,9 +17,9 @@
     </gazebo>
     <gazebo reference="camera_link">
-        <material>Gazebo/Blue</material>
+        <material>Blue</material>
     </gazebo>
     <gazebo reference="chasis">
         <material>
-          bodyTexture
+            bodyTexture
         </material>
     </gazebo>

File: src/gazebo_pg/urdf/example_robot.urdf.xacro (robot description, xacro)
@@ -29,5 +29,7 @@
                 <box size="${body_length} ${body_width} ${body_height}"/>
             </geometry>
-            <material name="blue"/>
+            <material name="bodyTexture">
+                <color rgba="1 1 1 1"/>
+            </material>
         </visual>
         <collision>
